File: flyback-pcb/flyback.kicad_sch (KiCad schematic)
At the start: 11 parts, among them U1 CAP200DG

Commit message: Updated .gitignore and moved acdc to acdc sheet
Parts:
- removed C1: 47nF, symbol Device:C
- removed C2: 330nF, symbol Device:C
- removed L1: WE-LF_SMD_SH, WE-LF_SMD_SH:WE-LF_SMD_SH, symbol WE-LF_SMD_SH:WE-LF_SMD_SH
- removed L5: WE-LPCC, WE-LPCC:WE-LPCC_7448680140, symbol WE-LPCC:WE-LPCC
- removed R1, R2: 1M, symbol Device:R_Small_US
- removed R3, R4: 0ZCA0100FF2E, 0ZCA0100FF2E:RESC3216X125N, symbol 0ZCA0100FF2E:0ZCA0100FF2E
- removed RT1: MS32_50006, MS32_50006:THERM_MS32_50006, symbol MS32_50006:MS32_50006
- removed RV1: B88069X2701S102, B88069X2701S102:RESAD1540W100L790D820, symbol B88069X2701S102:B88069X2701S102
- removed U1: CAP200DG, Package_SO:SOIC-8_3.9x4.9mm_P1.27mm, symbol Power_Management:CAP200DG

Commit message: Update flyback.kicad_sch
found components
Parts:
- added U1: MIN1072M-TL, MINSOP-16A_PWI, symbol min1072m-tl:MIN1072M-TL
Changed lines of the file:
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@@
 	(generator_version "8.0")
 	(paper "A4")
+	(text_box "ERJ-8GEYJ395V"
+		(exclude_from_sim no)
+		(at 22.86 24.13 0)
+		(size 26.67 30.48)
+		(stroke
+			(width 0)
+			(type default)
+		)
+		(fill
+			(type none)
+		)
+		(effects
+			(font
+				(size 1.27 1.27)
+			)
+			(justify left top)
+		)
+	)
+	(symbol
+		(lib_id "min1072m-tl:MIN1072M-TL")
+		(at 71.12 106.68 0)
+		(unit 1)
+		(exclude_from_sim no)
+		(in_bom yes)
+		(on_board yes)
+		(dnp no)
+		(fields_autoplaced yes)
+		(property "Reference" "U1"
+			(at 91.44 96.52 0)
+			(effects
+				(font
+					(size 1.524 1.524)
+				)
+			)
+		)
+		(property "Value" "MIN1072M-TL"
+			(at 91.44 99.06 0)
+			(effects
+				(font
+					(size 1.524 1.524)
+				)
+			)
+		)
+		(property "Footprint" "MINSOP-16A_PWI"
+			(at 71.12 106.68 0)
+			(effects
+				(font
+					(size 1.27 1.27)
+					(italic yes)
+				)
+				(hide yes)
+			)
+		)
+		(property "Datasheet" "MIN1072M-TL"
+			(at 71.12 106.68 0)
+			(effects
+				(font
+					(size 1.27 1.27)
+					(italic yes)
+				)
+				(hide yes)
+			)
+		)
+		(property "Description" ""
+			(at 71.12 106.68 0)
+			(effects
+				(font
+					(size 1.27 1.27)
+				)
+				(hide yes)
+			)
+		)
+		(pin "16"
+		)
+		(pin "10"
+		)
+		(pin "9"
+		)
+		(pin "5"
+		)
+		(pin "1"
+		)
+		(pin "3"
+		)
+		(pin "8"
+		)
+		(pin "11"
+		)
+		(pin "2"
+		)
+		(pin "6"
+		)
+		(pin "7"
+		)
+		(pin "4"
+		)
+		(instances
+			(project ""
+				(path "/ed7c0781-0d20-4118-b9de-6cfbb6417a17/16bd232e-5ea0-49a5-b25c-6403c4d2754c"
+					(reference "U1")
+					(unit 1)
+				)
+			)
+		)
+	)
 )
