File: flyback-pcb/flyback.kicad_sch (KiCad schematic)
At the start: 10 parts, among them U1 CAP200DG, U2 CAP200DG

Commit message: day2part2
Parts:
- removed L1, L2: L, symbol Device:L
- removed L3, L4: 230µH, symbol Device:L
- removed U2: CAP200DG, Package_SO:SOIC-8_3.9x4.9mm_P1.27mm, symbol Power_Management:CAP200DG
- added L5: WE-LPCC, WE-LPCC:WE-LPCC_7448680140, symbol WE-LPCC:WE-LPCC
Connections:
- net at R2.1: no longer C1.2
- net at C1.1: now also L5.3; no longer R1.1
- net at C2.1: now also L5.4
- net at C2.2: now also L5.1
- new net: C1.2, L5.2

Commit message: nearlyDone
Parts:
- added L1: WE-LF_SMD_SH, WE-LF_SMD_SH:WE-LF_SMD_SH, symbol WE-LF_SMD_SH:WE-LF_SMD_SH
- added R3, R4: 0ZCA0100FF2E, 0ZCA0100FF2E:RESC3216X125N, symbol 0ZCA0100FF2E:0ZCA0100FF2E
- added RT1: MS32_50006, MS32_50006:THERM_MS32_50006, symbol MS32_50006:MS32_50006
- added RV1: B88069X2701S102, B88069X2701S102:RESAD1540W100L790D820, symbol B88069X2701S102:B88069X2701S102
Connections:
- net at R2.1: now also C1.2, L5.2, L1.1
- net at C1.1, L5.3: now also R1.1, L1.4
- net at C2.2, L5.1: now also R3.2, RT1.2, RV1.2
- net at C2.1, L5.4: now also R3.1, R4.2, RV1.1
Other:
- moved on the sheet: C1, C2, L5, R1, R2, U1
