File: flyback-pcb/ac-dc.kicad_sch (KiCad schematic)
At the start: 0 parts

Commit message: Updated .gitignore and moved acdc to acdc sheet
Parts:
- added C3: 330nF, symbol Device:C
- added C4: 47nF, symbol Device:C
- added L2: WE-LPCC, WE-LPCC:WE-LPCC_7448680140, symbol WE-LPCC:WE-LPCC
- added L3: WE-LF_SMD_SH, WE-LF_SMD_SH:WE-LF_SMD_SH, symbol WE-LF_SMD_SH:WE-LF_SMD_SH
- added R5, R6: 0ZCA0100FF2E, 0ZCA0100FF2E:RESC3216X125N, symbol 0ZCA0100FF2E:0ZCA0100FF2E
- added R7, R8: 1M, symbol Device:R_Small_US
- added RT2: MS32_50006, MS32_50006:THERM_MS32_50006, symbol MS32_50006:MS32_50006
- added RV2: B88069X2701S102, B88069X2701S102:RESAD1540W100L790D820, symbol B88069X2701S102:B88069X2701S102
- added U2: CAP200DG, Package_SO:SOIC-8_3.9x4.9mm_P1.27mm, symbol Power_Management:CAP200DG
Connections:
- new net: C3.1, L2.4, R5.2, R6.1, RV2.1
- new net: C3.2, L2.1, R6.2, RT2.2, RV2.2
- new net: C4.2, L2.2, L3.1, R8.1
- new net: R8.2, U2.6, U2.7
- new net: C4.1, L2.3, L3.4, R7.1
- new net: R7.2, U2.2, U2.3

Commit message: nearNearDone
Parts:
- removed R5, R6: 0ZCA0100FF2E, 0ZCA0100FF2E:RESC3216X125N, symbol 0ZCA0100FF2E:0ZCA0100FF2E
- removed RT2: MS32_50006, MS32_50006:THERM_MS32_50006, symbol MS32_50006:MS32_50006
- added BR1: TT10M-13, TT10M_DIO, symbol 2024-10-22_12-55-56:TT10M-13
- added R1: SL08 20002, SL08 20002_AMT, symbol 2024-10-22_14-27-07:SL08_20002
- added R2, R3: 0ZCA0100FF2E, 0ZCA0100FF2E:RESC3216X125N, symbol 0ZCA0100FF2E:0ZCA0100FF2E
Connections:
- net at C3.1, L2.4, RV2.1: now also R2.2, R3.2
- net at C3.2, L2.1, RV2.2: now also R1.2, R3.1
- net at L3.2: now also BR1.3
- net at L3.3: now also BR1.4

Commit message: fuseChange
Parts:
- removed R2, R3: 0ZCA0100FF2E, 0ZCA0100FF2E:RESC3216X125N, symbol 0ZCA0100FF2E:0ZCA0100FF2E
- added F1, F2: Polyfuse, symbol Device:Polyfuse
Connections:
- net at C3.1, L2.4, RV2.1: now also F1.2, F2.2
- net at C3.2, L2.1, R1.2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: now also F2.1

Commit message: variable resistor
Parts:
- removed F2: Polyfuse, symbol Device:Polyfuse
- added R2: R_Variable_US, symbol Device:R_Variable_US
Connections:
- net at C3.2, L2.1, R1.2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: now also R2.2
- net at C3.1, F1.2, L2.4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: now also R2.1
Changed lines of the file:
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@@
-	)
-	(symbol
-		(lib_id "Device:Polyfuse")
-		(at 113.03 92.71 180)
-		(unit 1)
-		(exclude_from_sim no)
-		(in_bom yes)
-		(on_board yes)
-		(dnp no)
-		(fields_autoplaced yes)
-		(property "Reference" "F2"
-			(at 115.57 91.4399 0)
-			(effects
-				(font
-					(size 1.27 1.27)
-				)
-				(justify right)
-			)
-		)
-		(property "Value" "Polyfuse"
-			(at 115.57 93.9799 0)
-			(effects
-				(font
-					(size 1.27 1.27)
-				)
-				(justify right)
-			)
-		)
-		(property "Footprint" ""
-			(at 111.76 87.63 0)
-			(effects
-				(font
-					(size 1.27 1.27)
-				)
-				(justify left)
-				(hide yes)
-			)
-		)
-		(property "Datasheet" "~"
-			(at 113.03 92.71 0)
-			(effects
-				(font
-					(size 1.27 1.27)
-				)
-				(hide yes)
-			)
-		)
-		(property "Description" "Resettable fuse, polymeric positive temperature coefficient"
-			(at 113.03 92.71 0)
-			(effects
-				(font
-					(size 1.27 1.27)
-				)
-				(hide yes)
-			)
-		)
-		(pin "1"
-		)
-		(pin "2"
-		)
-		(instances
-			(project "flyback-pcb"
-				(path "/ed7c0781-0d20-4118-b9de-6cfbb6417a17/f6f3b632-57ee-4368-8954-2ac72372b096"
-					(reference "F2")
-					(unit 1)
-				)
-			)
-		)
 	)
 	(symbol
@@
 					(unit 1)
 				)
+			)
+		)
+	)
+	(symbol
+		(lib_id "Device:R_Variable_US")
+		(at 113.03 92.71 0)
+		(unit 1)
+		(exclude_from_sim no)
+		(in_bom yes)
+		(on_board yes)
+		(dnp no)
+		(fields_autoplaced yes)
+		(property "Reference" "R2"
+			(at 116.84 91.4018 0)
+			(effects
+				(font
+					(size 1.27 1.27)
+				)
+				(justify left)
+			)
+		)
+		(property "Value" "R_Variable_US"
+			(at 116.84 93.9418 0)
+			(effects
+				(font
+					(size 1.27 1.27)
+				)
+				(justify left)
+			)
+		)
+		(property "Footprint" ""
+			(at 111.252 92.71 90)
+			(effects
+				(font
+					(size 1.27 1.27)
+				)
+				(hide yes)
+			)
+		)
+		(property "Datasheet" "~"
+			(at 113.03 92.71 0)
+			(effects
+				(font
+					(size 1.27 1.27)
+				)
+				(hide yes)
+			)
+		)
+		(property "Description" "Variable resistor, US symbol"
+			(at 113.03 92.71 0)
+			(effects
+				(font
+					(size 1.27 1.27)
+				)
+				(hide yes)
+			)
+		)
+		(pin "1"
+		)
+		(pin "2"
+		)
+		(instances
+			(project ""
+				(path "/ed7c0781-0d20-4118-b9de-6cfbb6417a17/f6f3b632-57ee-4368-8954-2ac72372b096"
+					(reference "R2")
+					(unit 1)
+				)

Commit message: Re-done ac-dc
Parts:
- renumbered C4 to C22, C3 to C25, RV2 to G1, L2 to L1, L3 to L2, R7 to R21, R8 to R22, R2 to R23, R1 to R24, BR1 to RC1
Connections:
- net N: now reaches R24.1
- net HV_GND: now reaches RC1.1
- net HV+: now reaches RC1.2
- net L: now reaches F1.1
- no-connect marks 0 -> 4
Other:
- note added: "2 STAGE EMI FILTER"
- note added: "AC_FILTER_CAP_DISCHARGER"
- note added: "FULL BRIDGE RECT"
- note added: "INRUSH LIMITER"
- note added: "RESETABLE FUSE"
- note added: "SURGE ARRESTER GDT"
